File: Schaltung/Schaltung.sch (KiCad schematic (older format))
At the start: 37 parts, among them J1 Elektroden, Q1 IRF4905, Q2 IRF4905, Q3 IRF1404, Q4 IRF1404, Q5 IRF1404, Q6 IRF1404, Q7 IRF1404, SW1 SW_Push, U1 TC4420

Commit message: new annotation
Parts:
- gave numbers to parts that had none: 20
Changed lines of the file:
@@
 $EndDescr
 $Comp
-L +12V #PWR1
+L +12V #PWR7
 U 1 1 5ABA1DC9
 P 800 2850
-F 0 "#PWR1" H 800 2700 50  0001 C CNN
+F 0 "#PWR7" H 800 2700 50  0001 C CNN
 F 1 "+12V" H 800 2990 50  0000 C CNN
 F 2 "" H 800 2850 50  0001 C CNN
@@
 $EndComp
 $Comp
-L GND #PWR4
+L GND #PWR3
 U 1 1 5ABA1DDD
 P 5950 1900
-F 0 "#PWR4" H 5950 1650 50  0001 C CNN
+F 0 "#PWR3" H 5950 1650 50  0001 C CNN
 F 1 "GND" H 5950 1750 50  0000 C CNN
 F 2 "" H 5950 1900 50  0001 C CNN
@@
 $EndComp
 $Comp
-L GND #PWR6
+L GND #PWR19
 U 1 1 5ABA3862
 P 9850 5950
-F 0 "#PWR6" H 9850 5700 50  0001 C CNN
+F 0 "#PWR19" H 9850 5700 50  0001 C CNN
 F 1 "GND" H 9850 5800 50  0000 C CNN
 F 2 "" H 9850 5950 50  0001 C CNN
@@
 $EndComp
 $Comp
-L GND #PWR3
+L GND #PWR4
 U 1 1 5ABA420C
 P 8900 1950
-F 0 "#PWR3" H 8900 1700 50  0001 C CNN
+F 0 "#PWR4" H 8900 1700 50  0001 C CNN
 F 1 "GND" H 8900 1800 50  0000 C CNN
 F 2 "" H 8900 1950 50  0001 C CNN
@@
 $EndComp
 $Comp
-L GND #PWR5
+L GND #PWR15
 U 1 1 5ABA514E
 P 9750 5050
-F 0 "#PWR5" H 9750 4800 50  0001 C CNN
+F 0 "#PWR15" H 9750 4800 50  0001 C CNN
 F 1 "GND" H 9750 4900 50  0000 C CNN
 F 2 "" H 9750 5050 50  0001 C CNN
@@
 $EndComp
 $Comp
-L LM358 U?
+L LM358 U5
 U 1 1 5ABBDDF8
 P 4600 4200
-F 0 "U?" H 4600 4400 50  0000 L CNN
+F 0 "U5" H 4600 4400 50  0000 L CNN
 F 1 "LM358" H 4600 4000 50  0000 L CNN
 F 2 "" H 4600 4200 50  0001 C CNN
@@
 $EndComp
 $Comp
-L LM358 U?
+L LM358 U5
 U 2 1 5ABBDE43
 P 5500 4200
-F 0 "U?" H 5500 4400 50  0000 L CNN
+F 0 "U5" H 5500 4400 50  0000 L CNN
 F 1 "LM358" H 5500 4000 50  0000 L CNN
 F 2 "" H 5500 4200 50  0001 C CNN
@@
 $EndComp
 $Comp
-L ARDUINO_NANO ARDUINO?
+L ARDUINO_NANO ARDUINO1
 U 1 1 5ABBE3AC
 P 3150 6800
-F 0 "ARDUINO?" H 3150 7650 70  0000 C CNN
+F 0 "ARDUINO1" H 3150 7650 70  0000 C CNN
 F 1 "ARDUINO_NANO" V 3150 6800 70  0000 C CNN
 F 2 "" H 3150 6800 60  0000 C CNN
@@
 $EndComp
 $Comp
-L AP1117-50 U?
+L AP1117-50 U3
 U 1 1 5ABBEE6C
 P 1500 3300
-F 0 "U?" H 1350 3425 50  0000 C CNN
+F 0 "U3" H 1350 3425 50  0000 C CNN
 F 1 "AP1117-50" H 1500 3425 50  0000 L CNN
 F 2 "TO_SOT_Packages_SMD:SOT-223-3Lead_TabPin2" H 1500 3500 50  0001 C CNN
@@
 $EndComp
 $Comp
-L CP C?
+L CP C6
 U 1 1 5ABBF129
 P 800 3450
-F 0 "C?" H 825 3550 50  0000 L CNN
+F 0 "C6" H 825 3550 50  0000 L CNN
 F 1 "100µF" H 825 3350 50  0000 L CNN
 F 2 "" H 838 3300 50  0001 C CNN
@@
 $EndComp
 $Comp
-L CP C?
+L CP C7
 U 1 1 5ABBF390
 P 2550 3450
-F 0 "C?" H 2575 3550 50  0000 L CNN
+F 0 "C7" H 2575 3550 50  0000 L CNN
 F 1 "4F" H 2575 3350 50  0000 L CNN
 F 2 "" H 2588 3300 50  0001 C CNN
@@
 $EndComp
 $Comp
-L C C?
+L C C8
 U 1 1 5ABBF396
 P 2950 3450
-F 0 "C?" H 2975 3550 50  0000 L CNN
+F 0 "C8" H 2975 3550 50  0000 L CNN
 F 1 "100nF" H 2975 3350 50  0000 L CNN
 F 2 "" H 2988 3300 50  0001 C CNN
@@
 $EndComp
 $Comp
-L GND #PWR?
+L GND #PWR11
 U 1 1 5ABBF39C
 P 1500 3800
-F 0 "#PWR?" H 1500 3550 50  0001 C CNN
+F 0 "#PWR11" H 1500 3550 50  0001 C CNN
 F 1 "GND" H 1500 3650 50  0000 C CNN
 F 2 "" H 1500 3800 50  0001 C CNN
@@
 $EndComp
 $Comp
-L D D?
+L D D1
 U 1 1 5ABBF3DD
 P 800 3000
-F 0 "D?" H 800 3100 50  0000 C CNN
+F 0 "D1" H 800 3100 50  0000 C CNN
 F 1 "D" H 800 2900 50  0000 C CNN
 F 2 "" H 800 3000 50  0001 C CNN
@@
 $EndComp
 $Comp
-L R R?
+L R R4
 U 1 1 5ABBF965
 P 2150 3300
-F 0 "R?" V 2230 3300 50  0000 C CNN
+F 0 "R4" V 2230 3300 50  0000 C CNN
 F 1 "5" V 2150 3300 50  0000 C CNN
 F 2 "" V 2080 3300 50  0001 C CNN
@@
 $EndComp
 $Comp
-L +12V #PWR?
+L +12V #PWR1
 U 1 1 5ABBFF82
 P 5200 800
-F 0 "#PWR?" H 5200 650 50  0001 C CNN
+F 0 "#PWR1" H 5200 650 50  0001 C CNN
 F 1 "+12V" H 5200 940 50  0000 C CNN
 F 2 "" H 5200 800 50  0001 C CNN
@@
 $EndComp
 $Comp
-L +5V #PWR?
+L +5V #PWR8
 U 1 1 5ABC1D69
 P 2950 3100
-F 0 "#PWR?" H 2950 2950 50  0001 C CNN
+F 0 "#PWR8" H 2950 2950 50  0001 C CNN
 F 1 "+5V" H 2950 3240 50  0000 C CNN
 F 2 "" H 2950 3100 50  0001 C CNN
@@
 $EndComp
 $Comp
-L +12V #PWR?
+L +12V #PWR6
 U 1 1 5ABC1E37
 P 4850 2700
-F 0 "#PWR?" H 4850 2550 50  0001 C CNN
+F 0 "#PWR6" H 4850 2550 50  0001 C CNN
 F 1 "+12V" H 4850 2840 50  0000 C CNN
 F 2 "" H 4850 2700 50  0001 C CNN
@@
 $EndComp
 $Comp
-L GND #PWR?
+L GND #PWR12
 U 1 1 5ABC1E93
 P 5400 4550
-F 0 "#PWR?" H 5400 4300 50  0001 C CNN
+F 0 "#PWR12" H 5400 4300 50  0001 C CNN
 F 1 "GND" H 5400 4400 50  0000 C CNN
 F 2 "" H 5400 4550 50  0001 C CNN
@@
 $EndComp
 $Comp
-L +12V #PWR?
+L +12V #PWR2
 U 1 1 5ABC2427
 P 9600 1350
-F 0 "#PWR?" H 9600 1200 50  0001 C CNN
+F 0 "#PWR2" H 9600 1200 50  0001 C CNN
 F 1 "+12V" H 9600 1490 50  0000 C CNN
 F 2 "" H 9600 1350 50  0001 C CNN
@@
 MosfetDriver1
 $Comp
-L C C?
+L C C1
 U 1 1 5ABC3E74
 P 4550 3000
-F 0 "C?" H 4575 3100 50  0000 L CNN
+F 0 "C1" H 4575 3100 50  0000 L CNN
 F 1 "100nF" H 4575 2900 50  0000 L CNN
 F 2 "" H 4588 2850 50  0001 C CNN
@@
 $EndComp
 $Comp
-L GND #PWR?
+L GND #PWR9
 U 1 1 5ABC4092
 P 4550 3200
-F 0 "#PWR?" H 4550 2950 50  0001 C CNN
+F 0 "#PWR9" H 4550 2950 50  0001 C CNN
 F 1 "GND" H 4550 3050 50  0000 C CNN
 F 2 "" H 4550 3200 50  0001 C CNN
@@
 $EndComp
 $Comp
-L +5V #PWR?
+L +5V #PWR18
 U 1 1 5ABC48A3
 P 4100 5900
-F 0 "#PWR?" H 4100 5750 50  0001 C CNN
+F 0 "#PWR18" H 4100 5750 50  0001 C CNN
 F 1 "+5V" H 4100 6040 50  0000 C CNN
 F 2 "" H 4100 5900 50  0001 C CNN
@@
 $EndComp
 $Comp
-L GND #PWR?
+L GND #PWR20
 U 1 1 5ABC49B9
 P 1550 6200
-F 0 "#PWR?" H 1550 5950 50  0001 C CNN
+F 0 "#PWR20" H 1550 5950 50  0001 C CNN
 F 1 "GND" H 1550 6050 50  0000 C CNN
 F 2 "" H 1550 6200 50  0001 C CNN
@@
 $EndComp
 $Comp
-L R R?
+L R R3
 U 1 1 5ABC5566
 P 7200 1750
-F 0 "R?" V 7280 1750 50  0000 C CNN
+F 0 "R3" V 7280 1750 50  0000 C CNN
 F 1 "12" V 7200 1750 50  0000 C CNN
 F 2 "" V 7130 1750 50  0001 C CNN
@@
 $EndComp
 $Comp
-L BUZ11 Q?
+L BUZ11 Q8
 U 1 1 5ABC566D
 P 7300 2250
-F 0 "Q?" H 7550 2325 50  0000 L CNN
+F 0 "Q8" H 7550 2325 50  0000 L CNN
 F 1 "IRF1404" H 7550 2250 50  0000 L CNN
 F 2 "TO_SOT_Packages_THT:TO-220_Vertical" H 7550 2175 50  0001 L CIN
@@
 $EndComp
 $Comp
-L GND #PWR?
+L GND #PWR5
 U 1 1 5ABC573B
 P 7200 2550
-F 0 "#PWR?" H 7200 2300 50  0001 C CNN
+F 0 "#PWR5" H 7200 2300 50  0001 C CNN
 F 1 "GND" H 7200 2400 50  0000 C CNN
 F 2 "" H 7200 2550 50  0001 C CNN
@@
 $EndComp
 $Comp
-L MIC4427 U?
+L MIC4427 U4
 U 1 1 5ABC5C85
 P 8450 3600
-F 0 "U?" H 8350 4100 50  0000 R CNN
+F 0 "U4" H 8350 4100 50  0000 R CNN
 F 1 "TC4420" H 8350 4000 50  0000 R CNN
 F 2 "" H 8450 3300 50  0001 C CNN
@@
 $EndComp
 $Comp
-L MIC4427 U?
+L MIC4427 U2
 U 1 1 5ABC5D36
 P 9400 2750
-F 0 "U?" H 9300 3250 50  0000 R CNN
+F 0 "U2" H 9300 3250 50  0000 R CNN
 F 1 "TC4420" H 9300 3150 50  0000 R CNN
 F 2 "" H 9400 2450 50  0001 C CNN
@@
 welding
 $Comp
-L CP C?
+L CP C5
 U 1 1 5ABC7754
 P 5200 3000
-F 0 "C?" H 5225 3100 50  0000 L CNN
+F 0 "C5" H 5225 3100 50  0000 L CNN
 F 1 "4,7µF" H 5225 2900 50  0000 L CNN
 F 2 "" H 5238 2850 50  0001 C CNN
@@
 $EndComp
 $Comp
-L GND #PWR?
+L GND #PWR10
 U 1 1 5ABC7A2A
 P 5200 3200
-F 0 "#PWR?" H 5200 2950 50  0001 C CNN
+F 0 "#PWR10" H 5200 2950 50  0001 C CNN
 F 1 "GND" H 5200 3050 50  0000 C CNN
 F 2 "" H 5200 3200 50  0001 C CNN
@@
 MosfetDriver3
 $Comp
-L R R?
+L R R5
 U 1 1 5ABC9350
 P 4900 5150
-F 0 "R?" V 4980 5150 50  0000 C CNN
+F 0 "R5" V 4980 5150 50  0000 C CNN
 F 1 "15k" V 4900 5150 50  0000 C CNN
 F 2 "" V 4830 5150 50  0001 C CNN
@@
 $EndComp
 $Comp
-L R R?
+L R R6
 U 1 1 5ABC9458
 P 5800 5150
-F 0 "R?" V 5880 5150 50  0000 C CNN
+F 0 "R6" V 5880 5150 50  0000 C CNN
 F 1 "15k" V 5800 5150 50  0000 C CNN
 F 2 "" V 5730 5150 50  0001 C CNN
@@
 $EndComp
 $Comp
-L R R?
+L R R7
 U 1 1 5ABC94FF
 P 4700 5500
-F 0 "R?" V 4780 5500 50  0000 C CNN
+F 0 "R7" V 4780 5500 50  0000 C CNN
 F 1 "10k" V 4700 5500 50  0000 C CNN
 F 2 "" V 4630 5500 50  0001 C CNN
@@
 $EndComp
 $Comp
-L R R?
+L R R8
 U 1 1 5ABC9599
 P 5600 5500
-F 0 "R?" V 5680 5500 50  0000 C CNN
+F 0 "R8" V 5680 5500 50  0000 C CNN
 F 1 "10k" V 5600 5500 50  0000 C CNN
 F 2 "" V 5530 5500 50  0001 C CNN
@@
 $EndComp
 $Comp
-L GND #PWR?
+L GND #PWR16
 U 1 1 5ABC9759
 P 4550 5650
-F 0 "#PWR?" H 4550 5400 50  0001 C CNN
+F 0 "#PWR16" H 4550 5400 50  0001 C CNN
 F 1 "GND" H 4550 5500 50  0000 C CNN
 F 2 "" H 4550 5650 50  0001 C CNN
@@
 $EndComp
 $Comp
-L GND #PWR?
+L GND #PWR17
 U 1 1 5ABC97CD
 P 5450 5650
-F 0 "#PWR?" H 5450 5400 50  0001 C CNN
+F 0 "#PWR17" H 5450 5400 50  0001 C CNN
 F 1 "GND" H 5450 5500 50  0000 C CNN
 F 2 "" H 5450 5650 50  0001 C CNN
@@
 Connection ~ 5800 5500
 $Comp
-L SSD1306 U?
+L SSD1306 U6
 U 1 1 5ABCA032
 P 2250 4800
-F 0 "U?" H 3600 5400 60  0000 R TNN
+F 0 "U6" H 3600 5400 60  0000 R TNN
 F 1 "SSD1306" H 900 5400 60  0000 L TNN
 F 2 "" H 2250 4800 60  0001 C CNN
@@
 	1550 5150 1550 4800
 $Comp
-L +5V #PWR?
+L +5V #PWR14
 U 1 1 5ABCA611
 P 650 5050
-F 0 "#PWR?" H 650 4900 50  0001 C CNN
+F 0 "#PWR14" H 650 4900 50  0001 C CNN
 F 1 "+5V" H 650 5190 50  0000 C CNN
 F 2 "" H 650 5050 50  0001 C CNN
@@
 	650  5100 650  5050
 $Comp
-L GND #PWR?
+L GND #PWR13
 U 1 1 5ABCA75F
 P 2350 4950
-F 0 "#PWR?" H 2350 4700 50  0001 C CNN
+F 0 "#PWR13" H 2350 4700 50  0001 C CNN
 F 1 "GND" H 2350 4800 50  0000 C CNN
 F 2 "" H 2350 4950 50  0001 C CNN
@@
 	2350 4800 2350 4950
 $Comp
-L Rotary_Encoder_Switch SW?
+L Rotary_Encoder_Switch SW2
 U 1 1 5ABCA868
 P 4900 7250
-F 0 "SW?" H 4900 7510 50  0000 C CNN
+F 0 "SW2" H 4900 7510 50  0000 C CNN
 F 1 "Rotary_Encoder_Switch" H 4900 6990 50  0000 C CNN
 F 2 "" H 4800 7410 50  0001 C CNN
@@
 	4600 7250 4350 7250
 $Comp
-L GND #PWR?
+L GND #PWR21
 U 1 1 5ABCB1F0
 P 5900 7350
-F 0 "#PWR?" H 5900 7100 50  0001 C CNN
+F 0 "#PWR21" H 5900 7100 50  0001 C CNN
 F 1 "GND" H 5900 7200 50  0000 C CNN
 F 2 "" H 5900 7350 50  0001 C CNN

Commit message: add Leds, Buzzer, 1 inverted Mosfet Driver, 16V input
Parts:
- removed D1, D2: D, symbol D
- removed R4: 5, symbol R
- added BZ1: Buzzer, symbol Buzzer
- added C1: 0,47µF, symbol CP
- added C10: 100nF, symbol C
- added D1, D2: D_Schottky, symbol D_Schottky
- added D3: green, symbol LED
- added D4: red, symbol LED
- added R8, R9: 510, symbol R
- added U1: Step Up, TO_SOT_Packages_SMD:SOT-223-3Lead_TabPin2, symbol AP1117-50
- added U2: L7810, TO_SOT_Packages_SMD:SOT-223-3Lead_TabPin2, symbol AP1117-50
- C2: value 100µF -> 1000µF
- C4: value 2F -> 1F
- C7: renamed from C6; value 100µF -> 0,47µF
- C8: renamed from C7; value 4F -> 47µF
- R1: renamed from R2; value 0,86 -> 5
- R3: renamed from R1; value 0,86 -> 5
- R4: renamed from R5; value 15k -> 22k
- R5: renamed from R6; value 15k -> 22k
- U3: renamed from U2; value TC4420 -> TC4429; symbol MIC4427 -> MIC4426
- U4: renamed from U3; value AP1117-50 -> LM7805
- renumbered C1 to C5, C5 to C6, C8 to C9, Q8 to Q3, Q3 to Q4, Q4 to Q5, Q5 to Q6, Q6 to Q7, Q7 to Q8, R3 to R2, R7 to R6, R8 to R7, U4 to U5, U5 to U6, U1 to U7, U6 to U8
Connections:
- net +12V: now also D1.2 (A), D2.2 (A), U1.3 (VI); no longer C5.1, C6.1, Q1.2 (S), Q2.2 (S), U6.8 (V+), U6.8 (V+)
- net +5V: now also U4.2 (VO), C10.1
- net GND: now also C7.2, BZ1.1 (-), C1.2, D3.1 (K), D4.1 (K), U1.1 (GND), U2.1 (GND)
- net at C4.1, J1.1 (Pin_1), R1.1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: now also R3.1
- net at R1.2: now also Q1.3 (D), Q2.3 (D), R3.2; no longer R3.1
- net +15V: now reaches C2.1, C3.1, U3.6 (V+), U5.6 (V+), U7.6 (V+)
- net +15V: now also C5.1, C6.1, Q1.2 (S), Q2.2 (S), U6.8 (V+), U6.8 (V+), U1.2 (VO), U2.2 (VO)
- net at ARDUINO1.10 (D7): now also R9.1
- net at ARDUINO1.12 (D9): now also BZ1.2 (+)
- net at ARDUINO1.13 (D10): now also R8.1
- net at ARDUINO1.29 (GND): now also C10.2
- net at C7.1, U4.3 (VI): now also D2.1 (K)
- new net: C1.1, D1.1 (K), U2.3 (VI)
- new net: D3.2 (A), R8.2
- new net: D4.2 (A), R9.2
Other:
- note added: "10V Regulator for Mosfet Gates"
- note added: "150W Step Up Converter"
- note added: "5V Regulator for Arduino, IC and display"
- moved on the sheet: C7, C8, C9, R1, R3, U4
